Commit message: updated till gazebo spawn

File: description/robot_core.xacro (robot description, xacro)
@@ -1,10 +1,10 @@
 <?xml version="1.0"?>
-<robot xmlns:xacro="http://www.ros.org/wiki/xacro"  name="robot">
-<xacro:include filename="inertial_macros.xacro"/>
+<robot xmlns:xacro="http://www.ros.org/wiki/xacro" >
+    <xacro:include filename="inertial_macros.xacro"/>
     <material name="white">
-        <color rgba="1 1 1 1"/>
+        <color rgba="1 1 1 1" />
     </material>
     <material name="orange">
-        <color rgba="1 0.3 0.3 1"/>
+        <color rgba="1 0.3 0.1 1"/>
     </material>
     <material name="blue">
@@ -14,7 +14,8 @@
         <color rgba="0 0 0 1"/>
     </material>
+    <!-- BASE LINK -->
     <link name="base_link">
     </link>
-<!-- BASE LINK-->
+    <!-- CHASSIS LINK -->
     <joint name="chassis_joint" type="fixed">
         <parent link="base_link"/>
@@ -22,5 +23,4 @@
         <origin xyz="-0.1 0 0"/>
     </joint>
-<!-- CHASSIS LINKS-->
     <link name="chassis">
         <visual>
@@ -37,18 +37,20 @@
             </geometry>
         </collision>
-       <xacro:inertial_box mass="0.5" x="0.3" y="0.3" z="0.15">
+        <xacro:inertial_box mass="0.5" x="0.3" y="0.3" z="0.15">
             <origin xyz="0.15 0 0.075" rpy="0 0 0"/>
         </xacro:inertial_box>
     </link>
-<!--LEFT WHEEL LINKS-->
+    <gazebo reference="chassis">
+        <material>Gazebo/white</material>
+    </gazebo>
+    <!-- LEFT WHEEL LINK -->
     <joint name="left_wheel_joint" type="continuous">
         <parent link="base_link"/>
         <child link="left_wheel"/>
-        <origin xyz="0 0.175 0" rpy="-${pi/2} 0 0"/>
+        <origin xyz="0 0.175 0" rpy="-${pi/2} 0 0" />
         <axis xyz="0 0 1"/>
     </joint>
     <link name="left_wheel">
         <visual>
-            <origin xyz="0 0 0.05"/>
             <geometry>
                 <cylinder radius="0.05" length="0.04"/>
@@ -57,23 +59,24 @@
         </visual>
         <collision>
-            <origin xyz="0 0 0.05"/>
             <geometry>
                 <cylinder radius="0.05" length="0.04"/>
             </geometry>
         </collision>
-        <xacro:inertial_cylinder mass="0.1" radius="0.05" length="0.04">
+        <xacro:inertial_cylinder mass="0.1" length="0.04" radius="0.05">
             <origin xyz="0 0 0" rpy="0 0 0"/>
         </xacro:inertial_cylinder>
     </link>
-<!--RIGHT WHEEL LINKS-->
+    <gazebo reference="left_wheel">
+        <material>Gazebo/blue</material>
+    </gazebo>
+    <!-- RIGHT WHEEL LINK -->
     <joint name="right_wheel_joint" type="continuous">
         <parent link="base_link"/>
         <child link="right_wheel"/>
-        <origin xyz="0 -0.175 0" rpy="${pi/2} 0 0"/>
+        <origin xyz="0 -0.175 0" rpy="${pi/2} 0 0" />
         <axis xyz="0 0 -1"/>
     </joint>
     <link name="right_wheel">
         <visual>
-            <origin xyz="0 0 0.05"/>
             <geometry>
                 <cylinder radius="0.05" length="0.04"/>
@@ -82,20 +85,22 @@
         </visual>
         <collision>
-            <origin xyz="0 0 0.05"/>
             <geometry>
                 <cylinder radius="0.05" length="0.04"/>
             </geometry>
         </collision>
-        <xacro:inertial_cylinder mass="0.1" radius="0.05" length="0.04">
+        <xacro:inertial_cylinder mass="0.1" length="0.04" radius="0.05">
             <origin xyz="0 0 0" rpy="0 0 0"/>
         </xacro:inertial_cylinder>
     </link>
-<!-- CASTOR WHEEL LINK-->
-    <joint name="castor_wheel_joint" type="fixed">
+    <gazebo reference="right_wheel">
+        <material>Gazebo/blue</material>
+    </gazebo>
+    <!-- CASTER WHEEL LINK -->
+    <joint name="caster_wheel_joint" type="fixed">
         <parent link="chassis"/>
-        <child link="castor_wheel"/>
+        <child link="caster_wheel"/>
         <origin xyz="0.24 0 0"/>
     </joint>
-    <link name="castor_wheel">
+    <link name="caster_wheel">
         <visual>
             <geometry>
@@ -113,3 +118,6 @@
         </xacro:inertial_sphere>
     </link>
+    <gazebo reference="caster_wheel">
+        <material>Gazebo/black</material>
+    </gazebo>
 </robot>
