Commit message: changed files to adpat to new ignition gazebo

File: description/gazebo_control.xacro (robot description, xacro)
@@ -1,4 +1,29 @@
 <?xml version="1.0"?>
-<robot xmlns:xacro="http://www.ros.org/wiki/xacro"  name="robot">
-    <gazebo></>
+<robot xmlns:xacro="http://www.ros.org/wiki/xacro">
+    <gazebo>
+        <plugin name="gz::sim::systems::DiffDrive" filename="gz-sim-diff-drive-system">
+            <!-- Wheel Information -->
+            <left_joint>left_wheel_joint</left_joint>
+            <right_joint>right_wheel_joint</right_joint>
+            <wheel_separation>0.297</wheel_separation>
+            <wheel_radius>0.033</wheel_radius>
+            <!-- Limits -->
+            <!-- <max_wheel_torque>200</max_wheel_torque> -->
+            <max_linear_acceleration>0.33</max_linear_acceleration>
+            <!-- Input -->
+            <topic>cmd_vel</topic>
+            <!-- Output -->
+            <frame_id>odom</frame_id>
+            <child_frame_id>base_link</child_frame_id>
+            <odom_topic>odom</odom_topic>
+            <odom_publisher_frequency>30</odom_publisher_frequency>
+            <tf_topic>/tf</tf_topic>
+        </plugin>
+        <plugin filename="gz-sim-joint-state-publisher-system"
+            name="gz::sim::systems::JointStatePublisher">
+            <topic>joint_states</topic>
+            <joint_name>left_wheel_joint</joint_name>
+            <joint_name>right_wheel_joint</joint_name>
+       </plugin>
+    </gazebo>
 </robot>

File: description/robot_core.xacro (robot description, xacro)
@@ -41,7 +41,7 @@
         </xacro:inertial_box>
     </link>
-    <gazebo reference="chassis">
-        <material>Gazebo/white</material>
-    </gazebo>
+    <!-- <gazebo reference="chassis">
+        <material>Gazebo/White</material>
+    </gazebo> -->
     <!-- LEFT WHEEL LINK -->
     <joint name="left_wheel_joint" type="continuous">
@@ -67,7 +67,7 @@
         </xacro:inertial_cylinder>
     </link>
-    <gazebo reference="left_wheel">
-        <material>Gazebo/blue</material>
-    </gazebo>
+    <!-- <gazebo reference="left_wheel">
+        <material>Gazebo/Blue</material>
+    </gazebo> -->
     <!-- RIGHT WHEEL LINK -->
     <joint name="right_wheel_joint" type="continuous">
@@ -93,7 +93,7 @@
         </xacro:inertial_cylinder>
     </link>
-    <gazebo reference="right_wheel">
-        <material>Gazebo/blue</material>
-    </gazebo>
+    <!-- <gazebo reference="right_wheel">
+        <material>Gazebo/Blue</material>
+    </gazebo> -->
     <!-- CASTER WHEEL LINK -->
     <joint name="caster_wheel_joint" type="fixed">
@@ -118,6 +118,32 @@
         </xacro:inertial_sphere>
     </link>
+    <!-- <gazebo reference="caster_wheel">
+        <material>Gazebo/Black</material>
+        <mu1 value="0.001"/>
+        <mu2 value="0.001"/>
+    </gazebo> -->
+    <gazebo reference="chassis">
+        <material>
+            <ambient>1 1 1 1</ambient>     <!-- white -->
+            <diffuse>1 1 1 1</diffuse>
+        </material>
+    </gazebo>
+    <gazebo reference="left_wheel">
+    <material>
+        <ambient>0 0 1 1</ambient>     <!-- blue -->
+        <diffuse>0 0 1 1</diffuse>
+    </material>
+    </gazebo>
+    <gazebo reference="right_wheel">
+    <material>
+        <ambient>0 0 1 1</ambient>
+        <diffuse>0 0 1 1</diffuse>
+    </material>
+    </gazebo>
     <gazebo reference="caster_wheel">
-        <material>Gazebo/black</material>
+    <material>
+        <ambient>0 0 0 1</ambient>     <!-- black -->
+        <diffuse>0 0 0 1</diffuse>
+    </material>
     </gazebo>
 </robot>
