Commit message: added lidar and similated it on ign

File: description/robot.urdf.xacro (robot description, xacro)
@@ -3,3 +3,4 @@
 <xacro:include filename="robot_core.xacro"/>
 <xacro:include filename="gazebo_control.xacro"/>
+ <xacro:include filename="lidar.xacro" />
 </robot>

File: description/robot_core.xacro (robot description, xacro)
@@ -15,4 +15,16 @@
     <color rgba="0 0 0 1"/>
   </material>
+  <material name="green">
+  <color rgba="0 1 0 1" />
+</material>
+<material name="yellow">
+  <color rgba="1 1 0 1" />
+</material>
+<material name="red">
+  <color rgba="1 0 0 1" />
+</material>
+<material name="violet">
+  <color rgba="0.5 0 0.5 1" />
+</material>
   <!-- Base Link -->
   <link name="base_link" />
